File: pcb/full_n64_ctrl_board.kicad_pcb (KiCad board)
At the start: 2 copper layers, 135 x 54 mm, 32 parts, among them J1 Conn_01x02_Male, J10 Conn_01x02_Male, J11 Conn_01x02_Male, J12 Conn_01x02_Male, J13 Conn_01x02_Male, J14 Conn_01x02_Male, J15 Conn_01x02_Male, J16 Conn_01x02_Male, J17 Conn_01x02_Male, J18 Conn_01x02_Male, J19 Conn_01x04_Male, J2 Conn_01x02_Male, J20 Conn_01x04_Male, J21 Conn_01x02_Male, J22 Conn_01x02_Male, J23 Conn_01x15_Male, J24 Conn_01x15_Male, J25 Conn_01x15_Male, J26 Conn_01x15_Male, J27 Conn_01x15_Male, J28 Conn_01x15_Male, J29 Conn_01x02_Male, J3 Conn_01x02_Male, J30 Conn_01x02_Male, J31 Conn_01x02_Male, J4 Conn_01x02_Male, J5 Conn_01x02_Male, J6 Conn_01x02_Male, J7 Conn_01x02_Male, J8 Conn_01x02_Male, J9 Conn_01x02_Male

Commit message: update files
Parts:
- removed J31: Conn_01x02_Male, Connector_JST:JST_PH_S2B-PH-K_1x02_P2.00mm_Horizontal
- J21: footprint Connector_PinHeader_2.54mm:PinHeader_1x02_P2.54mm_Vertical -> full_n64_ctrl_board:2_pad
- J22: footprint full_n64_ctrl_board:2_pad -> Connector_PinHeader_2.54mm:PinHeader_1x02_P2.54mm_Vertical
- J23, J28: value Conn_01x15_Male -> Conn_01x13_Male; footprint Connector_PinHeader_2.54mm:PinHeader_1x15_P2.54mm_Vertical -> full_n64_ctrl_board:13_pad
- J24, J27: value Conn_01x15_Male -> Conn_01x13_Male; footprint Connector_PinHeader_2.54mm:PinHeader_1x15_P2.54mm_Vertical -> Connector_PinHeader_2.54mm:PinHeader_1x13_P2.54mm_Vertical
- J25, J26: value Conn_01x15_Male -> Conn_01x13_Male; footprint full_n64_ctrl_board:15_pad -> Connector_PinHeader_2.54mm:PinHeader_1x13_P2.54mm_Vertical
- moved J22 38.6 mm to (32.2, 79.7), turned to 40 degrees
- moved J21 36.3 mm to (27.6, 74.6), turned to 310 degrees
- moved J27 21.4 mm to (79.2, 54.4), turned to 80 degrees
- moved J26 17.4 mm to (78.2, 59.2), turned to 80 degrees
- moved J24 17.1 mm to (82.0, 36.6), turned to 80 degrees
- moved J23 15.2 mm to (80.6, 44.1), turned to 350 degrees
- moved J28 13.2 mm to (79.7, 51.5), turned to 350 degrees
- moved J25 9.39 mm to (81.2, 41.2), turned to 80 degrees
- moved J18 1.08 mm to (94.0, 32.4)
- moved J20 0.75 mm to (114.3, 77.8)
Connections:
- J21 pad 1: Net-(J21-Pad1) -> VCC
- J22 pad 1: Net-(J21-Pad1) -> VCC
- J23 pad 1: Net-(J21-Pad1) -> Net-(J23-Pad1)
- J23 pad 11: Net-(J16-Pad2) -> Net-(J13-Pad2)
- J23 pad 12: Net-(J19-Pad2) -> Net-(J14-Pad2)
- J23 pad 13: Net-(J19-Pad4) -> VCC
- J23 pad 2: GND -> Net-(J23-Pad2)
- J23 pad 4: Net-(J10-Pad2) -> Net-(J23-Pad4)
- J23 pad 5: Net-(J23-Pad5) -> Net-(J18-Pad1)
- J23 pad 7: Net-(J1-Pad2) -> Net-(J12-Pad2)
- J23 pad 8: Net-(J2-Pad2) -> Net-(J23-Pad8)
- J23 pad 9: Net-(J23-Pad9) -> Net-(J15-Pad2)
- J24 pad 1: Net-(J21-Pad1) -> Net-(J23-Pad1)
- J24 pad 11: Net-(J16-Pad2) -> Net-(J13-Pad2)
- J24 pad 12: Net-(J19-Pad2) -> Net-(J14-Pad2)
- J24 pad 13: Net-(J19-Pad4) -> VCC
- J24 pad 2: GND -> Net-(J23-Pad2)
- J24 pad 4: Net-(J10-Pad2) -> Net-(J23-Pad4)
- J24 pad 5: Net-(J23-Pad5) -> Net-(J18-Pad1)
- J24 pad 7: Net-(J1-Pad2) -> Net-(J12-Pad2)
- J24 pad 8: Net-(J2-Pad2) -> Net-(J23-Pad8)
- J24 pad 9: Net-(J23-Pad9) -> Net-(J15-Pad2)
- J25 pad 1: Net-(J21-Pad1) -> Net-(J23-Pad1)
- J25 pad 11: Net-(J16-Pad2) -> Net-(J13-Pad2)
- J25 pad 12: Net-(J19-Pad2) -> Net-(J14-Pad2)
- J25 pad 13: Net-(J19-Pad4) -> VCC
- J25 pad 2: GND -> Net-(J23-Pad2)
- J25 pad 4: Net-(J10-Pad2) -> Net-(J23-Pad4)
- J25 pad 5: Net-(J23-Pad5) -> Net-(J18-Pad1)
- J25 pad 7: Net-(J1-Pad2) -> Net-(J12-Pad2)
- J25 pad 8: Net-(J2-Pad2) -> Net-(J23-Pad8)
- J25 pad 9: Net-(J23-Pad9) -> Net-(J15-Pad2)
- J26 pad 1: VCC -> GND
- J26 pad 10: Net-(J13-Pad2) -> Net-(J19-Pad2)
- J26 pad 11: Net-(J12-Pad2) -> Net-(J26-Pad11)
- J26 pad 12: Net-(J26-Pad12) -> Net-(J19-Pad4)
- J26 pad 13: Net-(J26-Pad13) -> Net-(J11-Pad2)
- J26 pad 2: GND -> Net-(J10-Pad2)
- J26 pad 5: Net-(J18-Pad1) -> Net-(J1-Pad2)
- J26 pad 6: Net-(J26-Pad6) -> Net-(J2-Pad2)
- J26 pad 9: Net-(J15-Pad2) -> Net-(J16-Pad2)
- J27 pad 1: VCC -> GND
- J27 pad 10: Net-(J13-Pad2) -> Net-(J19-Pad2)
- J27 pad 11: Net-(J12-Pad2) -> Net-(J26-Pad11)
- J27 pad 12: Net-(J26-Pad12) -> Net-(J19-Pad4)
- J27 pad 13: Net-(J26-Pad13) -> Net-(J11-Pad2)
- J27 pad 2: GND -> Net-(J10-Pad2)
- J27 pad 5: Net-(J18-Pad1) -> Net-(J1-Pad2)
- J27 pad 6: Net-(J26-Pad6) -> Net-(J2-Pad2)
- J27 pad 9: Net-(J15-Pad2) -> Net-(J16-Pad2)
- J28 pad 1: VCC -> GND
- J28 pad 10: Net-(J13-Pad2) -> Net-(J19-Pad2)
- J28 pad 11: Net-(J12-Pad2) -> Net-(J26-Pad11)
- J28 pad 12: Net-(J26-Pad12) -> Net-(J19-Pad4)
- J28 pad 13: Net-(J26-Pad13) -> Net-(J11-Pad2)
- J28 pad 2: GND -> Net-(J10-Pad2)
- J28 pad 5: Net-(J18-Pad1) -> Net-(J1-Pad2)
- J28 pad 6: Net-(J26-Pad6) -> Net-(J2-Pad2)
- J28 pad 9: Net-(J15-Pad2) -> Net-(J16-Pad2)
- J29 pad 1: Net-(J26-Pad3) -> Net-(J23-Pad2)
- J29 pad 2: Net-(J26-Pad4) -> Net-(J23-Pad3)
- J3 pad 2: Net-(J23-Pad6) -> Net-(J26-Pad4)
- J30 pad 1: Net-(J26-Pad3) -> Net-(J23-Pad2)
- J30 pad 2: Net-(J26-Pad4) -> Net-(J23-Pad3)
- J4 pad 2: Net-(J26-Pad15) -> Net-(J26-Pad8)
- J5 pad 2: Net-(J26-Pad15) -> Net-(J26-Pad8)
- J6 pad 2: Net-(J23-Pad9) -> Net-(J26-Pad7)
- J9 pad 2: Net-(J23-Pad5) -> Net-(J26-Pad3)
Routing:
- net Net-(J23-Pad2): track 0.00 -> 78.4 mm
- net VCC: track 495.4 -> 420.7 mm
- net Net-(J23-Pad6): track 73.5 -> 8.07 mm
- net Net-(J23-Pad3): track 9.61 -> 72.6 mm
- net Net-(J23-Pad9): track 56.6 -> 0.00 mm
- net Net-(J23-Pad10): track 123.0 -> 73.3 mm
- net Net-(J26-Pad7): track 10.0 -> 56.4 mm
- net Net-(J23-Pad5): track 41.6 -> 0.00 mm
- net Net-(J21-Pad1): track 40.3 -> 0.00 mm
- net Net-(J26-Pad8): track 10.0 -> 46.8 mm
- net Net-(J26-Pad15): track 35.3 -> 0.00 mm
- net Net-(J26-Pad3): track 63.0 -> 40.8 mm
- net GND: track 145.9 -> 128.3 mm
- net Net-(J2-Pad2): track 63.8 -> 74.0 mm
- net Net-(J15-Pad2): track 105.7 -> 95.7 mm
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Other:
- outline, holes or cut-outs redrawn
- board text added: "D0"
- board text added: "D16/Rx2"
- board text added: "D17/Tx2"
- board text added: "ESP32lite N64 Controller v0.1 SVF"
- board text added: "Ext 3.3v"
- board text removed: "D21"
- board text removed: "ESP32 N64 Controller Board v0.1 SVF"
- board text removed: "Ext Pwr"
- board text removed: "Power"
- board text removed: "Rx"
- board text removed: "Rx2"
- board text removed: "Tx"
- board text removed: "Tx2"
- board text removed: "Vin"

Commit message: update PCB, update button mapping, re-enable battery level setup
Parts:
- added R2: R, Resistor_THT:R_Axial_DIN0207_L6.3mm_D2.5mm_P7.62mm_Horizontal, F.Cu at (112.5, 69.7)
- moved J24 0.50 mm to (81.5, 36.6)
- moved J25 0.50 mm to (80.7, 41.2)
- moved J26 0.50 mm to (77.7, 59.2)
- moved J27 0.50 mm to (78.7, 54.4)
- moved J11 0.35 mm to (85.2, 70.3)
Connections:
- J23 pad 6: Net-(J23-Pad6) -> Net-(J16-Pad2)
- J24 pad 6: Net-(J23-Pad6) -> Net-(J16-Pad2)
- J25 pad 6: Net-(J23-Pad6) -> Net-(J16-Pad2)
- J26 pad 9: Net-(J16-Pad2) -> Net-(J26-Pad9)
- J27 pad 9: Net-(J16-Pad2) -> Net-(J26-Pad9)
- J28 pad 9: Net-(J16-Pad2) -> Net-(J26-Pad9)
Routing:
- net GND: track 128.3 -> 112.9 mm
- net Net-(J26-Pad9): track 0.00 -> 8.30 mm
- net Net-(J11-Pad2): track 34.7 -> 43.0 mm
- net Net-(J23-Pad6): track 8.07 -> 0.00 mm
- net Net-(J16-Pad2): track 42.1 -> 50.0 mm
- net VCC: track 420.7 -> 423.9 mm
- net Net-(J26-Pad3): track 40.8 -> 43.4 mm
- net Net-(J12-Pad2): track 68.6 -> 70.0 mm
- net Net-(J15-Pad2): track 95.7 -> 96.3 mm
- net Net-(J19-Pad4): track 29.8 -> 30.3 mm
- net Net-(J19-Pad2): track 30.1 -> 30.6 mm
Other:
- outline, holes or cut-outs redrawn
- board text added: "ESP32lite N64 Controller v0.2b SVF"
- board text added: "gnd"
- board text removed: "ESP32lite N64 Controller v0.1 SVF"

Commit message: Update with experimental PCB
Parts:
- removed J28: Conn_01x13_Male, full_n64_ctrl_board:13_pad
- removed J29: Conn_01x02_Male, Connector_PinHeader_2.54mm:PinHeader_1x02_P2.54mm_Vertical
- removed J30: Conn_01x02_Male, full_n64_ctrl_board:2_pad
- added C1: 4.7uF, Capacitor_SMD:C_1206_3216Metric_Pad1.33x1.80mm_HandSolder, F.Cu at (59.9, 58.9)
- added C10: 4.7uF, Capacitor_SMD:C_1206_3216Metric_Pad1.33x1.80mm_HandSolder, F.Cu at (91.6, 41.6)
- added C11: 4.7uF, Capacitor_SMD:C_1206_3216Metric_Pad1.33x1.80mm_HandSolder, F.Cu at (97.8, 61.6)
- added C12: 0.1uF, Capacitor_SMD:C_1206_3216Metric_Pad1.33x1.80mm_HandSolder, F.Cu at (91.6, 44.4)
- added C13: 0.1uF, Capacitor_SMD:C_1206_3216Metric_Pad1.33x1.80mm_HandSolder, B.Cu at (57.9, 51.1)
- added C14: 0.1uF, Capacitor_SMD:C_1206_3216Metric_Pad1.33x1.80mm_HandSolder, B.Cu at (58.6, 39.9)
- added C15: 7pF, Capacitor_SMD:C_1206_3216Metric_Pad1.33x1.80mm_HandSolder, F.Cu at (114.7, 46.4)
- added C16: 7pF, Capacitor_SMD:C_1206_3216Metric_Pad1.33x1.80mm_HandSolder, F.Cu at (114.7, 44.0)
- added C17: 47pF, Capacitor_SMD:C_1206_3216Metric_Pad1.33x1.80mm_HandSolder, F.Cu at (91.4, 50.5)
- added C18: 4.7uF, Capacitor_SMD:C_1206_3216Metric_Pad1.33x1.80mm_HandSolder, F.Cu at (113.0, 38.2)
- added C19: 0.1uF, Capacitor_SMD:C_1206_3216Metric_Pad1.33x1.80mm_HandSolder, F.Cu at (98.8, 40.4)
- added C2: 0.1uF/50V, Capacitor_SMD:C_1206_3216Metric_Pad1.33x1.80mm_HandSolder, F.Cu at (40.9, 72.3)
- added C3: 0.1uF/50V, Capacitor_SMD:C_1206_3216Metric_Pad1.33x1.80mm_HandSolder, F.Cu at (49.8, 62.1)
- added C4: 22uF, Capacitor_SMD:C_1206_3216Metric_Pad1.33x1.80mm_HandSolder, F.Cu at (99.6, 70.4)
- added C5: 47pF, Capacitor_SMD:C_1206_3216Metric_Pad1.33x1.80mm_HandSolder, F.Cu at (91.6, 34.4)
- added C7: 0.1uF, Capacitor_SMD:C_1206_3216Metric_Pad1.33x1.80mm_HandSolder, F.Cu at (99.6, 72.7)
- added C8: 0.1uF, Capacitor_SMD:C_1206_3216Metric_Pad1.33x1.80mm_HandSolder, F.Cu at (91.6, 39.2)
- added C9: 4.7uF, Capacitor_SMD:C_1206_3216Metric_Pad1.33x1.80mm_HandSolder, F.Cu at (65.2, 58.8)
- added D1: D_TVS, Diode_SMD:D_SOD-323_HandSoldering, F.Cu at (93.5, 32.2)
- added D2: D_Schottky, Diode_SMD:D_SOD-123F, F.Cu at (62.5, 58.8)
- added D3: D_TVS, Diode_SMD:D_SOD-323_HandSoldering, F.Cu at (93.5, 28.2)
- added D4: D_TVS, Diode_SMD:D_SOD-323_HandSoldering, F.Cu at (93.5, 30.2)
- added D5: PowerLED, LED_SMD:LED_1206_3216Metric_Pad1.42x1.75mm_HandSolder, F.Cu at (78.8, 36.6)
- added D6: ChargeLED, LED_SMD:LED_1206_3216Metric_Pad1.42x1.75mm_HandSolder, F.Cu at (81.9, 36.5)
- added D7: LEDOut, LED_SMD:LED_1206_3216Metric_Pad1.42x1.75mm_HandSolder, F.Cu at (84.8, 36.5)
- added JP1: PowerLEDJumper, Jumper:SolderJumper-2_P1.3mm_Bridged_RoundedPad1.0x1.5mm, F.Cu at (69.7, 43.4)
- added JP2rx: RXJumper, Jumper:SolderJumper-2_P1.3mm_Bridged_RoundedPad1.0x1.5mm, F.Cu at (112.5, 41.1)
- added JP3tx: TXJumper, Jumper:SolderJumper-2_P1.3mm_Bridged_RoundedPad1.0x1.5mm, F.Cu at (98.5, 50.6)
- added Q1: Q_PMOS_GSD, Package_TO_SOT_SMD:SOT-23_Handsoldering, F.Cu at (71.5, 56.3)
- added Q2: Q_NPN_BEC, Package_TO_SOT_SMD:SOT-23_Handsoldering, F.Cu at (84.5, 57.4)
- added Q3: Q_NPN_BEC, Package_TO_SOT_SMD:SOT-23_Handsoldering, F.Cu at (91.8, 57.1)
- added R10: 10k, Resistor_SMD:R_1206_3216Metric_Pad1.30x1.75mm_HandSolder, F.Cu at (72.5, 50.5)
- added R11: 10k, Resistor_SMD:R_1206_3216Metric_Pad1.30x1.75mm_HandSolder, F.Cu at (88.2, 57.2)
- added R12: 10k, Resistor_SMD:R_1206_3216Metric_Pad1.30x1.75mm_HandSolder, F.Cu at (75.8, 50.5)
- added R13: 10k, Resistor_SMD:R_1206_3216Metric_Pad1.30x1.75mm_HandSolder, F.Cu at (76.3, 63.7)
- added R14: 3.3k, Resistor_SMD:R_1206_3216Metric_Pad1.30x1.75mm_HandSolder, F.Cu at (81.1, 50.5)
- added R15: 3M, Resistor_SMD:R_1206_3216Metric_Pad1.30x1.75mm_HandSolder, F.Cu at (83.7, 50.5)
- added R16: 4.7M, Resistor_SMD:R_1206_3216Metric_Pad1.30x1.75mm_HandSolder, F.Cu at (86.5, 50.5)
- added R3: 10k, Resistor_SMD:R_1206_3216Metric_Pad1.30x1.75mm_HandSolder, F.Cu at (69.3, 50.5)
- added R4: 27, Resistor_SMD:R_1206_3216Metric_Pad1.30x1.75mm_HandSolder, F.Cu at (91.5, 36.7)
- added R5: 27, Resistor_SMD:R_1206_3216Metric_Pad1.30x1.75mm_HandSolder, F.Cu at (91.5, 47.2)
- added R7: 6.8M, Resistor_SMD:R_1206_3216Metric_Pad1.30x1.75mm_HandSolder, F.Cu at (114.5, 51.0)
- added SW1: SW_Push, Button_Switch_THT:SW_PUSH_6mm, F.Cu at (54.7, 49.0)
- added SW2: SW_Push, Button_Switch_THT:SW_PUSH_6mm, F.Cu at (55.4, 37.9)
- added U1: RT9080-33GJ5, Package_TO_SOT_SMD:TSOT-23-5_HandSoldering, F.Cu at (71.4, 60.2)
- added U2: FT231XS, Package_SO:SSOP-20_3.9x8.7mm_P0.635mm, F.Cu at (105.2, 43.9)
- added U4: MCP73831-2-OT, Package_TO_SOT_SMD:SOT-23-5_HandSoldering, F.Cu at (79.5, 57.5)
- added U5: ESP32-WROOM-32, RF_Module:ESP32-WROOM-32, F.Cu at (113.8, 65.5)
- added Y1: Crystal 32.768kHz, Crystal:Crystal_SMD_3215-2Pin_3.2x1.5mm, F.Cu at (114.7, 48.7)
- J1: value Conn_01x02_Male -> DpadLeftPad
- J10: value Conn_01x02_Male -> APad
- J11: value Conn_01x02_Male -> StartPad
- J12: value Conn_01x02_Male -> CleftPad
- J13: value Conn_01x02_Male -> CupPad
- J14: value Conn_01x02_Male -> CdownPad
- J15: value Conn_01x02_Male -> CrightPad
- J16: value Conn_01x02_Male -> ZHole; footprint Connector_PinHeader_2.54mm:PinHeader_1x02_P2.54mm_Vertical -> Connector_JST:JST_PH_S2B-PH-K_1x02_P2.00mm_Horizontal
- J17: value Conn_01x02_Male -> ZPad
- J18: value Conn_01x02_Male -> SignalLED; footprint LED_THT:LED_D5.0mm_Horizontal_O3.81mm_Z3.0mm -> Connector_PinHeader_2.54mm:PinHeader_1x02_P2.54mm_Vertical
- J19: value Conn_01x04_Male -> AnalogHole; footprint Connector_PinHeader_2.54mm:PinHeader_1x04_P2.54mm_Vertical -> Connector_JST:JST_PH_S4B-PH-K_1x04_P2.00mm_Horizontal
- J2: value Conn_01x02_Male -> DpadUpPad
- J20: value Conn_01x04_Male -> AnalogPad
- J21: value Conn_01x02_Male -> ExtPowerPad
- J22: value Conn_01x02_Male -> ExtPowerHole
- J23: value Conn_01x13_Male -> USB_B_Micro; footprint full_n64_ctrl_board:13_pad -> Connector_USB:USB_Micro-B_Amphenol_10118194_Horizontal
- J24: value Conn_01x13_Male -> ExtBatPad; footprint Connector_PinHeader_2.54mm:PinHeader_1x13_P2.54mm_Vertical -> full_n64_ctrl_board:2_pad
- J25: value Conn_01x13_Male -> ExtBatHole; footprint Connector_PinHeader_2.54mm:PinHeader_1x13_P2.54mm_Vertical -> Connector_PinHeader_2.54mm:PinHeader_1x02_P2.54mm_Vertical
- J26: value Conn_01x13_Male -> Battery_Jumper; footprint Connector_PinHeader_2.54mm:PinHeader_1x13_P2.54mm_Vertical -> Connector_JST:JST_PH_S2B-PH-K_1x02_P2.00mm_Horizontal
- J27: value Conn_01x13_Male -> ExtIO21; footprint Connector_PinHeader_2.54mm:PinHeader_1x13_P2.54mm_Vertical -> Connector_PinHeader_2.54mm:PinHeader_1x02_P2.54mm_Vertical
- J3: value Conn_01x02_Male -> DpadDownPad
- J4: value Conn_01x02_Male -> LtriggerHole; footprint Connector_PinHeader_2.54mm:PinHeader_1x02_P2.54mm_Vertical -> Connector_JST:JST_PH_S2B-PH-K_1x02_P2.00mm_Horizontal
- J5: value Conn_01x02_Male -> LtriggerPad
- J6: value Conn_01x02_Male -> DpadRightPad
- J7: value Conn_01x02_Male -> RtriggerHole; footprint Connector_PinHeader_2.54mm:PinHeader_1x02_P2.54mm_Vertical -> Connector_JST:JST_PH_S2B-PH-K_1x02_P2.00mm_Horizontal
- J8: value Conn_01x02_Male -> RtriggerPad
- J9: value Conn_01x02_Male -> BPad
- R1, R2: value R -> 10k; footprint Resistor_THT:R_Axial_DIN0207_L6.3mm_D2.5mm_P7.62mm_Horizontal -> Resistor_SMD:R_1206_3216Metric_Pad1.30x1.75mm_HandSolder
- moved J20 60.4 mm to (54.0, 74.0)
- moved J19 58.6 mm to (52.1, 76.2), turned to 0 degrees
- moved R2 49.6 mm to (66.8, 50.5)
- moved J26 26.2 mm to (71.0, 33.9), turned to 0 degrees
- moved J27 24.7 mm to (103.1, 50.7), turned to 90 degrees
- moved J23 19.1 mm to (84.8, 25.5), turned to 180 degrees
- moved J25 13.4 mm to (73.2, 30.1), turned to 270 degrees
- moved J5 11.0 mm to (128.7, 51.0), turned to 180 degrees
- moved J24 8.37 mm to (77.4, 29.3), turned to 270 degrees
- moved J18 7.21 mm to (101.2, 32.0), turned to 330 degrees
- moved J16 4.05 mm to (70.8, 72.0), turned to 180 degrees
- moved J7 3.30 mm to (45.2, 48.3), turned to 180 degrees
- moved J8 3.11 mm to (45.6, 51.0), turned to 180 degrees
- moved J4 3.02 mm to (128.6, 47.1), turned to 180 degrees
- moved R1 0.65 mm to (64.3, 50.5), turned to 90 degrees
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Connections:
- J1 pad 1: VCC -> VDD
- J1 pad 2: Net-(J1-Pad2) -> IO26
- J10 pad 1: VCC -> VDD
- J10 pad 2: Net-(J10-Pad2) -> IO12
- J11 pad 1: VCC -> VDD
- J11 pad 2: Net-(J11-Pad2) -> SENSOR_VP
- J12 pad 1: VCC -> VDD
- J12 pad 2: Net-(J12-Pad2) -> IO17
- J13 pad 1: VCC -> VDD
- J13 pad 2: Net-(J13-Pad2) -> IO19
- J14 pad 1: VCC -> VDD
- J14 pad 2: Net-(J14-Pad2) -> IO22
- J15 pad 1: VCC -> VDD
- J15 pad 2: Net-(J15-Pad2) -> IO18
- J16 pad 1: VCC -> VDD
- J16 pad 2: Net-(J16-Pad2) -> IO16
- J17 pad 1: VCC -> VDD
- J17 pad 2: Net-(J16-Pad2) -> IO16
- J18 pad 1: Net-(J18-Pad1) -> IO5
- J19 pad 1: VCC -> IO21
- J19 pad 2: Net-(J19-Pad2) -> IO34
- J19 pad 4: Net-(J19-Pad4) -> SENSOR_VN
- J2 pad 1: VCC -> VDD
- J2 pad 2: Net-(J2-Pad2) -> IO25
- J20 pad 1: VCC -> IO21
- J20 pad 2: Net-(J19-Pad2) -> IO34
- J20 pad 4: Net-(J19-Pad4) -> SENSOR_VN
- J21 pad 1: VCC -> VDD
- J22 pad 1: VCC -> VDD
- J23 pad 1: Net-(J23-Pad1) -> VBUS
- J23 pad 2: Net-(J23-Pad2) -> USB_DN
- J23 pad 3: Net-(J23-Pad3) -> USB_DP
- J23 pad 5: Net-(J18-Pad1) -> GND
- J23 pad 6: Net-(J16-Pad2) -> Net-(J23-Pad6)
- J24 pad 1: Net-(J23-Pad1) -> VBAT
- J24 pad 2: Net-(J23-Pad2) -> GND
- J25 pad 1: Net-(J23-Pad1) -> VBAT
- J25 pad 2: Net-(J23-Pad2) -> GND
- J26 pad 2: Net-(J10-Pad2) -> VBAT
- J27 pad 1: GND -> IO2
- J27 pad 2: Net-(J10-Pad2) -> GND
- J3 pad 1: VCC -> VDD
- J3 pad 2: Net-(J26-Pad4) -> IO27
- J4 pad 1: VCC -> VDD
- J4 pad 2: Net-(J26-Pad8) -> IO4
- J5 pad 1: VCC -> VDD
- J5 pad 2: Net-(J26-Pad8) -> IO4
- J6 pad 1: VCC -> VDD
- J6 pad 2: Net-(J26-Pad7) -> IO13
- J7 pad 1: VCC -> VDD
- J7 pad 2: Net-(J23-Pad10) -> IO23
- J8 pad 1: VCC -> VDD
- J8 pad 2: Net-(J23-Pad10) -> IO23
- J9 pad 1: VCC -> VDD
- J9 pad 2: Net-(J26-Pad3) -> IO14
- R2 pad 1: GND -> VBUS
- R2 pad 2: Net-(J11-Pad2) -> GND
Routing:
- net VCC: track 423.9 -> 0.00 mm
- net VDD: track 0.00 -> 401.0 mm, vias 0 -> 7
- net GND: track 112.9 -> 377.8 mm, vias 0 -> 11
- net VBUS: track 0.00 -> 152.1 mm, vias 0 -> 8
- net EN: track 0.00 -> 131.2 mm, vias 0 -> 7
- net IO34: track 0.00 -> 102.4 mm, vias 0 -> 4
- net Net-(J14-Pad2): track 98.2 -> 0.00 mm
- net IO12: track 0.00 -> 98.1 mm, vias 0 -> 7
- net SENSOR_VN: track 0.00 -> 97.7 mm, vias 0 -> 4
- net Net-(J15-Pad2): track 96.3 -> 0.00 mm
- net Net-(J13-Pad2): track 89.2 -> 0.00 mm
- net Net-(J1-Pad2): track 85.7 -> 0.00 mm
- net IO22: track 0.00 -> 84.6 mm, vias 0 -> 3
- net IO18: track 0.00 -> 84.1 mm, vias 0 -> 1
- net VBAT: track 0.00 -> 83.1 mm, vias 0 -> 5
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- added copper zone on B.Cu, net VDD
- removed copper zone on B.Cu, net VCC
Other:
- board size 135 x 54 mm -> 132.5 x 62 mm
- board text added: "32"
- board text added: "33"
- board text added: "Auto Prog"
- board text added: "Bat+"
- board text added: "Bat-/G"
- board text added: "ESP32direct N64 Controller v0.3 SVF"
- board text added: "Flash"
- board text added: "G"
- board text added: "IO2"
- board text added: "Reset"
- board text added: "Volt Supply"
- board text added: "chrg"
- board text added: "io"
- board text added: "out"
- board text added: "pwr"
- board text added: "usb/ serial"
- board text removed: "Aux"
- board text removed: "Aux (pwr control)"
- board text removed: "D0"
- board text removed: "D12"
- board text removed: "D13"
- board text removed: "D14"
- board text removed: "D15"
- board text removed: "D16/Rx2"
- board text removed: "D17/Tx2"
- board text removed: "D18"
- board text removed: "D19"
- board text removed: "D2"
- board text removed: "D22"
- board text removed: "D23"
- board text removed: "D25"
- board text removed: "D26"
- board text removed: "D27"
- board text removed: "D32"
- board text removed: "D33"
- board text removed: "D34"
- board text removed: "D35"
- board text removed: "D4"
- board text removed: "D5"
- board text removed: "ESP32lite N64 Controller v0.2b SVF"
- board text removed: "En"
- board text removed: "Gnd"
- board text removed: "ONout"
- board text removed: "SWin"
- board text removed: "Vn"
- board text removed: "Vp"
